Commit message: we had added rgb-camera on turtlebot, and it finally worked, but I wanted to replace it with rgb-d camera

File: src/smart_cane_sim/smart_cane_sim/urdf/turtlebot3_burger.urdf (robot description, URDF)
Before this commit: robot turtlebot3_burger, 7 links, 6 joints
Links:
- added link camera_link, mass 0.1; collision box size=0.04 0.04 0.03; visual box size=0.04 0.04 0.03
Joints:
- added joint camera_joint: type fixed, parent base_link, child camera_link, origin xyz=0 0 0.25 rpy=0 0 0
